File: hardware/1590b/podal_1590b.kicad_sch (KiCad schematic)
At the start: 56 parts, among them J1 Guitar in, J2 fsw pin 1, J3 fsw pin 2, J4 fsw pin 4, J5 fsw pin 5, J6 fsw pin 6, J7 Left out, J8 Right out, J9 fsw pin 3, SW1 Switch 1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

Commit message: Compressor working with sensible led output
Parts:
- BT1: footprint Connector_BarrelJack:BarrelJack_Horizontal_centre_negative -> Connector_Wire:SolderWire-0.25sqmm_1x02_P4.2mm_D0.65mm_OD1.7mm
- C1: footprint Capacitor_THT:C_Radial_D10.0mm_H16.0mm_P5.00mm -> Capacitor_THT:C_Radial_D5.0mm_H11.0mm_P2.00mm
- J1, J7, J8: footprint Connector_Audio:Jack_6.35mm_Neutrik_NRJ6HM-1_Horizontal -> Connector_Wire:SolderWire-0.25sqmm_1x01_D0.65mm_OD2mm
- J2, J3, J4, J5, J6, J9: footprint Connector_Wire:SolderWire-0.75sqmm_1x01_D1.25mm_OD3.5mm -> Connector_Wire:SolderWire-0.25sqmm_1x01_D0.65mm_OD2mm
- SW1, SW2: footprint Connector_Wire:SolderWire-0.75sqmm_1x02_P7mm_D1.25mm_OD3.5mm -> Connector_Wire:SolderWire-0.15sqmm_1x02_P4mm_D0.5mm_OD1.5mm
Changed lines of the file:
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@@
     (title "DaisyPdal")
     (date "2024-04-25")
-    (rev "0.2")
+    (rev "0.3")
   )
   (junction (at 259.461 66.421) (diameter 0) (color 0 0 0 0)
@@
       (effects (font (size 1.27 1.27)) (justify left))
     )
-    (property "Footprint" "Connector_Wire:SolderWire-0.75sqmm_1x01_D1.25mm_OD3.5mm" (at 48.895 182.88 0)
+    (property "Footprint" "Connector_Wire:SolderWire-0.25sqmm_1x01_D0.65mm_OD2mm" (at 48.895 182.88 0)
       (effects (font (size 1.27 1.27)) hide)
     )
@@
       (effects (font (size 1.27 1.27)) (justify right))
     )
-    (property "Footprint" "Connector_Audio:Jack_6.35mm_Neutrik_NRJ6HM-1_Horizontal" (at 270.51 66.421 0)
+    (property "Footprint" "Connector_Wire:SolderWire-0.25sqmm_1x01_D0.65mm_OD2mm" (at 270.51 66.421 0)
       (effects (font (size 1.27 1.27)) hide)
     )
@@
       (effects (font (size 1.27 1.27)) (justify left))
     )
-    (property "Footprint" "Connector_Wire:SolderWire-0.75sqmm_1x01_D1.25mm_OD3.5mm" (at 273.812 34.544 0)
+    (property "Footprint" "Connector_Wire:SolderWire-0.25sqmm_1x01_D0.65mm_OD2mm" (at 273.812 34.544 0)
       (effects (font (size 1.27 1.27)) hide)
     )
@@
       (effects (font (size 1.27 1.27)))
     )
-    (property "Footprint" "Connector_Wire:SolderWire-0.75sqmm_1x02_P7mm_D1.25mm_OD3.5mm" (at 114.173 153.67 0)
+    (property "Footprint" "Connector_Wire:SolderWire-0.15sqmm_1x02_P4mm_D0.5mm_OD1.5mm" (at 114.173 153.67 0)
       (effects (font (size 1.27 1.27)) hide)
     )
@@
       (effects (font (size 1.27 1.27)) (justify left))
     )
-    (property "Footprint" "Connector_BarrelJack:BarrelJack_Horizontal_centre_negative" (at 18.415 169.926 90)
+    (property "Footprint" "Connector_Wire:SolderWire-0.25sqmm_1x02_P4.2mm_D0.65mm_OD1.7mm" (at 18.415 169.926 90)
       (effects (font (size 1.27 1.27)) hide)
     )
@@
       (effects (font (size 1.27 1.27)) (justify left))
     )
-    (property "Footprint" "Capacitor_THT:C_Radial_D10.0mm_H16.0mm_P5.00mm" (at 43.815 175.26 0)
+    (property "Footprint" "Capacitor_THT:C_Radial_D5.0mm_H11.0mm_P2.00mm" (at 43.815 175.26 0)
       (effects (font (size 1.27 1.27)) hide)
     )
@@
       (effects (font (size 1.27 1.27)) (justify left))
     )
-    (property "Footprint" "Connector_Wire:SolderWire-0.75sqmm_1x01_D1.25mm_OD3.5mm" (at 29.845 38.1 0)
+    (property "Footprint" "Connector_Wire:SolderWire-0.25sqmm_1x01_D0.65mm_OD2mm" (at 29.845 38.1 0)
       (effects (font (size 1.27 1.27)) hide)
     )
@@
       (effects (font (size 1.27 1.27)) (justify left))
     )
-    (property "Footprint" "Connector_Wire:SolderWire-0.75sqmm_1x01_D1.25mm_OD3.5mm" (at 32.893 50.8 0)
+    (property "Footprint" "Connector_Wire:SolderWire-0.25sqmm_1x01_D0.65mm_OD2mm" (at 32.893 50.8 0)
       (effects (font (size 1.27 1.27)) hide)
     )
@@
       (effects (font (size 1.27 1.27)))
     )
-    (property "Footprint" "Connector_Wire:SolderWire-0.75sqmm_1x02_P7mm_D1.25mm_OD3.5mm" (at 102.235 142.24 0)
+    (property "Footprint" "Connector_Wire:SolderWire-0.15sqmm_1x02_P4mm_D0.5mm_OD1.5mm" (at 102.235 142.24 0)
       (effects (font (size 1.27 1.27)) hide)
     )
@@
       (effects (font (size 1.27 1.27)))
     )
-    (property "Footprint" "Connector_Audio:Jack_6.35mm_Neutrik_NRJ6HM-1_Horizontal" (at 19.685 38.1 0)
+    (property "Footprint" "Connector_Wire:SolderWire-0.25sqmm_1x01_D0.65mm_OD2mm" (at 19.685 38.1 0)
       (effects (font (size 1.27 1.27)) hide)
     )
@@
       (effects (font (size 1.27 1.27)) (justify left))
     )
-    (property "Footprint" "Connector_Wire:SolderWire-0.75sqmm_1x01_D1.25mm_OD3.5mm" (at 258.064 100.711 0)
+    (property "Footprint" "Connector_Wire:SolderWire-0.25sqmm_1x01_D0.65mm_OD2mm" (at 258.064 100.711 0)
       (effects (font (size 1.27 1.27)) hide)
     )
@@
       (effects (font (size 1.27 1.27)) (justify left))
     )
-    (property "Footprint" "Connector_Wire:SolderWire-0.75sqmm_1x01_D1.25mm_OD3.5mm" (at 31.115 153.67 0)
+    (property "Footprint" "Connector_Wire:SolderWire-0.25sqmm_1x01_D0.65mm_OD2mm" (at 31.115 153.67 0)
       (effects (font (size 1.27 1.27)) hide)
     )
@@
       (effects (font (size 1.27 1.27)) (justify right))
     )
-    (property "Footprint" "Connector_Audio:Jack_6.35mm_Neutrik_NRJ6HM-1_Horizontal" (at 268.224 100.711 0)
-      (effects (font (size 1.27 1.27)) hide)
-    )
+    (property "Footprint" "Connector_Wire:SolderWire-0.25sqmm_1x01_D0.65mm_OD2mm" (at 268.224 100.711 0)
+      (effects (font (size 1.27 1.27)) hide)
+    )
