File: hardware/1590b/podal_1590b.kicad_pcb (KiCad board)
At the start: 2 copper layers, 54 x 60 mm, 56 parts, among them J1 Guitar in, J2 fsw pin 1, J3 fsw pin 2, J4 fsw pin 4, J5 fsw pin 5, J6 fsw pin 6, J7 Left out, J8 Right out, J9 fsw pin 3, SW1 Switch 1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

Commit message: Adjustments to silkscreen
Parts:
- moved J1 105.1 mm to (93.5, 52.9)
- moved J2 105.1 mm to (93.5, 56.9)
- moved J6 105.1 mm to (93.5, 61.0)
- moved J7 105.1 mm to (93.5, 65.0)
