File: hardware/1590bb/daisyPodal.kicad_sch (KiCad schematic)
At the start: 56 parts, among them J1 Guitar in, J2 fsw pin 1, J3 fsw pin 2, J4 fsw pin 4, J5 fsw pin 5, J6 fsw pin 6, J7 Left out, J8 Right out, J9 fsw pin 3, SW1 Switch 1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

Commit message: Reorganise hardware into enclosure size
Parts:
- BT1: footprint Connector_Wire:SolderWire-0.25sqmm_1x02_P4.2mm_D0.65mm_OD1.7mm -> Connector_BarrelJack:BarrelJack_Horizontal_centre_negative
- C1: footprint Capacitor_THT:C_Radial_D5.0mm_H11.0mm_P2.00mm -> Capacitor_THT:C_Radial_D10.0mm_H16.0mm_P5.00mm
- J1, J7, J8: footprint Connector_Wire:SolderWire-0.25sqmm_1x01_D0.65mm_OD2mm -> Connector_Audio:Jack_6.35mm_Neutrik_NRJ6HM-1_Horizontal
- J2, J3, J4, J5, J6, J9: footprint Connector_Wire:SolderWire-0.25sqmm_1x01_D0.65mm_OD2mm -> Connector_Wire:SolderWire-0.75sqmm_1x01_D1.25mm_OD3.5mm
- SW1, SW2: footprint Connector_Wire:SolderWire-0.15sqmm_1x02_P4mm_D0.5mm_OD1.5mm -> Connector_Wire:SolderWire-0.75sqmm_1x02_P7mm_D1.25mm_OD3.5mm
- U1: footprint Package_DIP:DIP-14_W7.62mm_Socket -> (none)
